File: rj_electronics/pcb/pcb_xyloauto/pcb_xyloauto.kicad_pcb (KiCad board)
At the start: 2 copper layers, 12 parts, among them J1 Conn_01x08_Pin, J2 Conn_01x08_Pin, J3 Conn_01x02_Pin, U1 Sparkfun_Pro_Micro, U2 ULN2803A, U3 LM317_TO-220

Commit message: nc
Parts:
- added J4: Barrel_Jack, Connector Barrel Jack - Community:BarrelJack_GCT_DCJ200-10-A_Horizontal, F.Cu at (194.4, 134.6)
- C1: footprint Capacitor_THT:CP_Radial_D10.0mm_P2.50mm -> Capacitor_THT:CP_Radial_D7.5mm_P2.50mm
- RV1: footprint Potentiometer_THT:Potentiometer_TT_P0915N -> Potentiometer_THT:Potentiometer_Bourns_3339P_Vertical
- moved J3 107.8 mm to (134.6, 134.6), turned to -90 degrees
- moved U2 82.3 mm to (76.2, 134.6), turned to 90 degrees
- moved U3 81.0 mm to (157.5, 142.2)
- moved J1 77.4 mm to (76.2, 142.2), turned to 90 degrees
- moved RV1 72.2 mm to (134.6, 129.5)
- moved C2 70.3 mm to (172.7, 139.7), turned to 180 degrees
- moved C1 69.7 mm to (182.9, 139.7)
- moved J2 65.9 mm to (101.6, 142.2)
- moved R1 61.9 mm to (137.2, 142.2)
- moved U1 60.4 mm to (71.1, 127.0)
- moved D2 59.3 mm to (142.2, 127.0)
- moved D1 55.9 mm to (142.2, 132.1), turned to 0 degrees
Connections:
- J2 pad 1: VIN -> VOUT
- J2 pad 2: VIN -> VOUT
- J2 pad 3: VIN -> VOUT
- J2 pad 4: VIN -> VOUT
- J2 pad 5: VIN -> VOUT
- J2 pad 6: VIN -> VOUT
- J2 pad 7: VIN -> VOUT
- J2 pad 8: VIN -> VOUT
- J3 pad 2: VIN -> VOUT
Routing:
- net VIN: track 170.8 -> 60.6 mm
- net Net-(U1-D2): track 82.1 -> 26.2 mm
- net Net-(U1-~D3): track 72.0 -> 26.5 mm
- net Net-(U1-D4/A6): track 65.7 -> 26.3 mm
- net Net-(U1-~D5): track 59.7 -> 26.3 mm
- net Net-(U1-~D6/A7): track 53.7 -> 26.3 mm
- net Net-(U1-D7): track 47.6 -> 26.3 mm
- net Net-(U1-D8/A8): track 41.6 -> 26.3 mm
- net Net-(D2-A): track 80.0 -> 64.7 mm
- net Net-(J1-Pin_8): track 6.34 -> 16.2 mm
- net Net-(J1-Pin_6): track 6.34 -> 16.2 mm
- net Net-(J1-Pin_7): track 6.34 -> 16.2 mm
- net Net-(J1-Pin_5): track 6.34 -> 16.2 mm
- net Net-(J1-Pin_4): track 6.34 -> 16.2 mm
- net Net-(J1-Pin_2): track 6.34 -> 16.2 mm
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Other:
- board outline added: 180 x 26 mm

Commit message: nc
Parts:
- J4: footprint Connector Barrel Jack - Community:BarrelJack_GCT_DCJ200-10-A_Horizontal -> Connector Barrel Jack - Community:BarrelJack_Wuerth_6941xx301002
- moved J4 143.2 mm to (52.0, 118.7), turned to -90 degrees
Routing:
- net VIN: track 60.6 -> 121.9 mm
- net GND: track 180.9 -> 165.7 mm
- net Net-(U1-~D9/A9): track 33.5 -> 26.2 mm
- net VOUT: track 159.1 -> 165.8 mm
- net Net-(D2-A): track 64.7 -> 67.5 mm
Other:
- board size 180 x 26 mm -> 180.3 x 36.2 mm

Commit message: nc
Parts:
- moved J2 56.1 mm to (157.5, 137.2)
- moved C2 35.9 mm to (208.3, 134.6)
- moved C1 34.5 mm to (210.9, 119.4)
- moved J1 28.4 mm to (88.9, 116.8)
- moved U3 25.9 mm to (182.9, 137.2)
- moved D1 18.0 mm to (160.0, 129.5)
- moved D2 17.0 mm to (157.5, 119.4)
- moved J4 16.6 mm to (68.6, 118.7)
- moved U2 13.0 mm to (88.9, 132.1)
- moved RV1 10.8 mm to (142.2, 121.9)
- moved J3 5.08 mm to (134.6, 129.5)
- moved R1 3.33 mm to (134.8, 139.9)
Routing:
- net Net-(D2-A): track 67.5 -> 106.8 mm
- net GND: track 165.7 -> 201.5 mm
- net VOUT: track 165.8 -> 197.9 mm
- net Net-(U1-D7): track 26.3 -> 40.1 mm
- net Net-(U1-~D9/A9): track 26.2 -> 39.9 mm
- net Net-(U1-~D6/A7): track 26.3 -> 40.1 mm
- net Net-(U1-~D5): track 26.3 -> 40.1 mm
- net Net-(U1-D2): track 26.2 -> 39.9 mm
- net Net-(U1-D8/A8): track 26.3 -> 40.1 mm
- net Net-(U1-D4/A6): track 26.3 -> 40.1 mm
- net Net-(U1-~D3): track 26.6 -> 40.3 mm
- net Net-(J1-Pin_1): track 16.2 -> 7.62 mm
- net Net-(J1-Pin_8): track 16.2 -> 7.62 mm
- net Net-(J1-Pin_7): track 16.2 -> 7.62 mm
- net Net-(J1-Pin_6): track 16.2 -> 7.62 mm
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Other:
- board size 180.3 x 36.2 mm -> 200 x 40 mm

Commit message: nc
Parts:
- moved J3 74.7 mm to (208.3, 116.8)
- moved RV1 38.1 mm to (180.3, 121.9)
- moved R1 32.3 mm to (157.5, 116.8)
- moved D2 30.6 mm to (188.0, 116.8)
- moved D1 28.4 mm to (188.0, 124.5)
- moved J1 24.0 mm to (101.6, 137.2)
- moved J4 20.4 mm to (48.2, 118.2)
- moved U2 18.3 mm to (73.7, 142.2)
- moved C1 17.0 mm to (218.5, 134.6)
- moved J2 12.7 mm to (144.8, 137.2)
- moved U3 8.03 mm to (190.5, 134.6)
- moved U1 2.64 mm to (68.5, 126.7)
Routing:
- net VOUT: track 197.9 -> 229.1 mm
- net Net-(D2-A): track 106.8 -> 76.9 mm
- net VIN: track 128.2 -> 155.8 mm
- net GND: track 201.5 -> 229.0 mm
- net Net-(J1-Pin_2): track 7.62 -> 32.4 mm
- net Net-(J1-Pin_5): track 7.62 -> 30.7 mm
- net Net-(J1-Pin_6): track 7.62 -> 30.7 mm
- net Net-(J1-Pin_7): track 7.62 -> 30.7 mm
- net Net-(J1-Pin_8): track 7.62 -> 30.7 mm
- net Net-(J1-Pin_3): track 7.62 -> 30.3 mm
- net Net-(J1-Pin_4): track 7.62 -> 29.3 mm
- net Net-(J1-Pin_1): track 7.62 -> 29.1 mm
- net Net-(U1-~D6/A7): track 40.1 -> 24.3 mm
- net Net-(U1-~D3): track 40.3 -> 24.6 mm
- net Net-(U1-~D9/A9): track 39.9 -> 25.1 mm
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
Commit message: nc
Parts:
- removed J2: Conn_01x08_Pin, Connector_PinSocket_2.54mm:PinSocket_1x08_P2.54mm_Vertical
- added J5: Screw_Terminal_01x08, TerminalBlock_Phoenix:TerminalBlock_Phoenix_PT-1,5-8-3.5-H_1x08_P3.50mm_Horizontal, F.Cu at (132.7, 119.4)
- J1: value Conn_01x08_Pin -> Screw_Terminal_01x08; footprint Connector_PinSocket_2.54mm:PinSocket_1x08_P2.54mm_Vertical -> TerminalBlock_Phoenix:TerminalBlock_Phoenix_PT-1,5-8-3.5-H_1x08_P3.50mm_Horizontal
- R1: footprint Resistor_THT:R_Axial_DIN0414_L11.9mm_D4.5mm_P15.24mm_Horizontal -> Resistor_THT:R_Axial_DIN0207_L6.3mm_D2.5mm_P10.16mm_Horizontal
- moved R1 104.1 mm to (53.3, 116.8)
- moved RV1 101.6 mm to (78.7, 121.9)
- moved J3 38.9 mm to (171.5, 129.5)
- moved U2 29.6 mm to (88.9, 116.8), turned to 0 degrees
- moved D2 22.8 mm to (165.2, 116.8)
- moved J1 17.9 mm to (103.5, 119.4), turned to 0 degrees
- moved D1 12.6 mm to (175.3, 123.7), turned to 180 degrees
Routing:
- net VOUT: track 229.1 -> 0.00 mm
- net GND: track 229.0 -> 0.00 mm
- net VIN: track 155.8 -> 0.00 mm
- net Net-(D2-A): track 76.9 -> 0.00 mm
- net Net-(J1-Pin_2): track 32.4 -> 0.00 mm
- net Net-(J1-Pin_5): track 30.7 -> 0.00 mm
- net Net-(J1-Pin_6): track 30.7 -> 0.00 mm
- net Net-(J1-Pin_7): track 30.7 -> 0.00 mm
- net Net-(J1-Pin_8): track 30.7 -> 0.00 mm
- net Net-(J1-Pin_3): track 30.3 -> 0.00 mm
- net Net-(J1-Pin_4): track 29.3 -> 0.00 mm
- net Net-(J1-Pin_1): track 29.1 -> 0.00 mm
- net Net-(U1-~D5): track 26.9 -> 0.00 mm
- net Net-(U1-D2): track 26.1 -> 0.00 mm
- net Net-(U1-D7): track 25.8 -> 0.00 mm
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
Commit message: nc
Parts:
- J3: value Conn_01x02_Pin -> VReg
- RV1: value R_Potentiometer_Trim -> Vreg RVar
- moved J3 110.2 mm to (61.8, 140.2), turned to 180 degrees
- moved R1 76.8 mm to (127.1, 138.3), turned to 90 degrees
- moved D1 41.4 mm to (134.2, 128.0), turned to -90 degrees
- moved D2 40.7 mm to (130.6, 138.2), turned to 90 degrees
- moved U3 25.4 mm to (165.1, 134.6)
- moved J4 19.0 mm to (48.3, 137.2)
- moved RV1 18.1 mm to (72.2, 138.7), turned to 90 degrees
- moved C2 18.0 mm to (190.5, 137.2), turned to 90 degrees
- moved U1 11.9 mm to (68.4, 114.8)
- moved U2 4.35 mm to (85.1, 114.7)
- moved C1 3.54 mm to (221.0, 132.1), turned to -90 degrees
- moved J1 2.50 mm to (103.4, 116.9)
- moved J5 2.50 mm to (132.7, 116.9)
Routing:
- net GND: track 0.00 -> 208.4 mm
- net VOUT: track 0.00 -> 205.5 mm
- net Net-(D2-A): track 0.00 -> 158.5 mm
- net VIN: track 0.00 -> 129.5 mm
- net Net-(J1-Pin_8): track 0.00 -> 41.7 mm
- net Net-(U1-D2): track 0.00 -> 41.0 mm
- net Net-(U1-~D3): track 0.00 -> 37.4 mm
- net Net-(J1-Pin_7): track 0.00 -> 37.1 mm
- net Net-(U1-D4/A6): track 0.00 -> 33.8 mm
- net Net-(J1-Pin_6): track 0.00 -> 32.6 mm
- net Net-(U1-~D5): track 0.00 -> 30.2 mm
- net Net-(J1-Pin_5): track 0.00 -> 28.0 mm
- net Net-(U1-~D6/A7): track 0.00 -> 26.6 mm
- net Net-(U1-D7): track 0.00 -> 24.1 mm
- net Net-(J1-Pin_4): track 0.00 -> 23.4 mm
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Other:
- board size 200 x 40 mm -> 200 x 37 mm

Commit message: nc
Parts:
- added D3: LED, LED_THT:LED_D5.0mm, F.Cu at (65.4, 140.1)
- added D4: LED, LED_THT:LED_D5.0mm, F.Cu at (104.6, 139.7)
- added D5: LED, LED_THT:LED_D5.0mm, F.Cu at (153.2, 139.8)
- added D6: LED, LED_THT:LED_D5.0mm, F.Cu at (196.1, 139.8)
- added R2: R, Resistor_THT:R_Axial_DIN0207_L6.3mm_D2.5mm_P10.16mm_Horizontal, F.Cu at (72.6, 142.2)
- added R3: R, Resistor_THT:R_Axial_DIN0207_L6.3mm_D2.5mm_P10.16mm_Horizontal, F.Cu at (112.3, 142.3)
- added R4: R, Resistor_THT:R_Axial_DIN0207_L6.3mm_D2.5mm_P10.16mm_Horizontal, F.Cu at (148.3, 142.3)
- added R5: R, Resistor_THT:R_Axial_DIN0207_L6.3mm_D2.5mm_P10.16mm_Horizontal, F.Cu at (192.2, 142.2)
- J3: value VReg -> Conn_01x02_Pin
- RV1: value Vreg RVar -> R_Potentiometer_Trim
- moved C2 22.9 mm to (213.4, 138.0), turned to 180 degrees
- moved RV1 17.3 mm to (55.5, 133.9), turned to 180 degrees
- moved D1 10.3 mm to (125.8, 134.1), turned to 0 degrees
- moved R1 9.40 mm to (136.0, 141.2), turned to 180 degrees
- moved J3 8.94 mm to (67.9, 133.7), turned to -90 degrees
- moved C1 5.75 mm to (221.3, 137.9), turned to 0 degrees
- moved D2 5.42 mm to (136.0, 137.7), turned to 180 degrees
Connections:
- U1 pad 17: unconnected-(U1-D18/A0-Pad17) -> LED1
- U1 pad 18: unconnected-(U1-D19/A1-Pad18) -> LED2
- U1 pad 19: unconnected-(U1-D20/A2-Pad19) -> LED3
- U1 pad 20: unconnected-(U1-D21/A3-Pad20) -> LED4
Routing:
- net LED4: track 0.00 -> 159.6 mm
- net LED3: track 0.00 -> 126.8 mm
- net LED2: track 0.00 -> 83.2 mm
- net LED1: track 0.00 -> 29.3 mm
- net VOUT: track 205.5 -> 224.9 mm
- net Net-(D2-A): track 158.5 -> 177.5 mm
- net Net-(D4-K): track 0.00 -> 8.94 mm
- net Net-(D3-K): track 0.00 -> 8.35 mm
- net GND: track 208.4 -> 214.8 mm
- net Net-(D5-K): track 0.00 -> 6.01 mm
- net Net-(D6-K): track 0.00 -> 4.89 mm
- net VIN: track 129.5 -> 126.9 mm

Commit message: nc
Parts:
- RV1: footprint Potentiometer_THT:Potentiometer_Bourns_3339P_Vertical -> Potentiometer_THT:Potentiometer_Bourns_3299W_Vertical
Routing:
- net VOUT: track 224.9 -> 0.00 mm
- net GND: track 214.8 -> 0.00 mm
- net Net-(D2-A): track 177.5 -> 0.00 mm
- net LED4: track 159.6 -> 0.00 mm
- net VIN: track 126.9 -> 0.00 mm
- net LED3: track 126.8 -> 0.00 mm
- net LED2: track 83.2 -> 0.00 mm
- net Net-(J1-Pin_8): track 41.7 -> 0.00 mm
- net Net-(U1-D2): track 41.0 -> 0.00 mm
- net Net-(U1-~D3): track 37.4 -> 0.00 mm
- net Net-(J1-Pin_7): track 37.1 -> 0.00 mm
- net Net-(U1-D4/A6): track 33.8 -> 0.00 mm
- net Net-(J1-Pin_6): track 32.6 -> 0.00 mm
- net Net-(U1-~D5): track 30.2 -> 0.00 mm
- net LED1: track 29.3 -> 0.00 mm
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