File: rj_electronics/pcb/pcb_xyloauto/pcb_xyloauto.kicad_pcb (KiCad board)
At the start: 2 copper layers, 200 x 37 mm, 21 parts, among them J1 Screw_Terminal_01x08, J3 Conn_01x02_Pin, J4 Barrel_Jack, J5 Screw_Terminal_01x08, U1 Sparkfun_Pro_Micro, U2 ULN2803A, U4 LM317_TO-220

Commit message: nc
Parts:
- removed J4: Barrel_Jack, Connector Barrel Jack - Community:BarrelJack_Wuerth_6941xx301002
- added J2: Conn_01x02_Pin, Connector_PinHeader_2.54mm:PinHeader_1x02_P2.54mm_Vertical, F.Cu at (219.5, 116.8)
- moved RV1 116.0 mm to (168.4, 120.5)
- moved C2 27.7 mm to (192.4, 119.1)
- moved C1 26.3 mm to (202.5, 118.5)
- moved U1 3.18 mm to (65.3, 114.2)
Connections:
- U1 pad 3: unconnected-(U1-GND-Pad3) -> GND
- U1 pad 4: unconnected-(U1-GND-Pad4) -> GND
Routing:
- net Net-(D2-A): track 174.9 -> 98.1 mm
- net VIN: track 125.0 -> 105.1 mm
- net LED2: track 63.7 -> 76.6 mm, vias 1 -> 0
- net VOUT: track 222.2 -> 213.4 mm
- net LED4: track 155.5 -> 162.9 mm
- net LED1: track 42.8 -> 35.6 mm
- net LED3: track 113.1 -> 118.2 mm
- net Net-(U1-D7): track 24.0 -> 27.9 mm
- net Net-(U1-D8/A8): track 20.5 -> 23.7 mm
- net Net-(U1-~D9/A9): track 18.0 -> 21.1 mm
- net GND: track 220.0 -> 223.2 mm
- net Net-(U1-~D6/A7): track 26.6 -> 29.7 mm
- net Net-(U1-D2): track 41.0 -> 43.9 mm
- net Net-(U1-~D3): track 37.4 -> 40.3 mm
- net Net-(U1-D4/A6): track 33.8 -> 36.7 mm
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