File: rj_electronics/pcb/pcb_xyloauto/pcb_xyloauto.kicad_sch (KiCad schematic)
At the start: 21 parts, among them J1 Screw_Terminal_01x08, J3 Conn_01x02_Pin, J4 Barrel_Jack, J5 Screw_Terminal_01x08, U1 Sparkfun_Pro_Micro, U2 ULN2803A, U4 LM317_TO-220

Commit message: nc
Connections:
- net GND: now also U1.3 (GND), U1.4 (GND)
- no-connect marks 10 -> 8

Commit message: nc
Parts:
- removed J4: Barrel_Jack, Connector Barrel Jack - Community:BarrelJack_Wuerth_6941xx301002, symbol Connector - Community:Barrel_Jack
- added J2: Conn_01x02_Pin, Connector_PinHeader_2.54mm:PinHeader_1x02_P2.54mm_Vertical, symbol Connector:Conn_01x02_Pin
Connections:
- net GND: now also J2.2 (Pin_2)
- net VIN: now also J2.1 (Pin_1)
Changed lines of the file:
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@@
+    (stroke (width 0) (type default))
+  )
+  (wire (pts (xy 160.02 30.48) (xy 162.56 30.48))
     (stroke (width 0) (type default))
   )
@@
     (stroke (width 0) (type default))
   )
-  (wire (pts (xy 160.02 33.02) (xy 165.1 33.02))
-    (stroke (width 0) (type default))
-  )
   (wire (pts (xy 219.71 99.06) (xy 219.71 101.6))
     (stroke (width 0) (type default))
@@
     (stroke (width 0) (type default))
   )
+  (wire (pts (xy 162.56 30.48) (xy 162.56 33.02))
+    (stroke (width 0) (type default))
+  )
   (wire (pts (xy 218.44 35.56) (xy 218.44 36.83))
     (stroke (width 0) (type default))
@@
     (stroke (width 0) (type default))
   )
+  (wire (pts (xy 162.56 33.02) (xy 165.1 33.02))
+    (stroke (width 0) (type default))
+  )
   (wire (pts (xy 97.79 138.43) (xy 167.64 138.43))
     (stroke (width 0) (type default))
@@
     (stroke (width 0) (type default))
   )
+  (wire (pts (xy 160.02 27.94) (xy 165.1 27.94))
+    (stroke (width 0) (type default))
+  )
   (wire (pts (xy 115.57 36.83) (xy 127 36.83))
     (stroke (width 0) (type default))
@@
   )
   (wire (pts (xy 55.88 106.68) (xy 55.88 107.95))
-    (stroke (width 0) (type default))
-  )
-  (wire (pts (xy 160.02 27.94) (xy 165.1 27.94))
     (stroke (width 0) (type default))
   )
@@
     )
   )
-  (symbol (lib_id "Connector - Community:Barrel_Jack") (at 152.4 30.48 0) (unit 1)
-    (in_bom yes) (on_board yes) (dnp no) (fields_autoplaced)
-    (property "Reference" "J4" (at 152.4 22.86 0)
+  (symbol (lib_id "Connector:Conn_01x02_Pin") (at 154.94 27.94 0) (unit 1)
+    (in_bom yes) (on_board yes) (dnp no) (fields_autoplaced)
+    (property "Reference" "J2" (at 155.575 24.13 0)
       (effects (font (size 1.27 1.27)))
     )
-    (property "Value" "Barrel_Jack" (at 152.4 25.4 0)
+    (property "Value" "Conn_01x02_Pin" (at 155.575 26.67 0)
       (effects (font (size 1.27 1.27)))
     )
-    (property "Footprint" "Connector Barrel Jack - Community:BarrelJack_Wuerth_6941xx301002" (at 153.67 31.496 0)
-      (effects (font (size 1.27 1.27)) hide)
-    )
-    (property "Datasheet" "~" (at 153.67 31.496 0)
-      (effects (font (size 1.27 1.27)) hide)
-    )
-    (pin "1")
-    (pin "2")
-    (instances
-      (project "pcb_xyloauto"
-        (path "/720c51e5-653f-4a9c-b040-f99d22f2970d"
-          (reference "J4") (unit 1)
-        )
-      )
+    (property "Footprint" "Connector_PinHeader_2.54mm:PinHeader_1x02_P2.54mm_Vertical" (at 154.94 27.94 0)
+      (effects (font (size 1.27 1.27)) hide)
+    )
+    (property "Datasheet" "~" (at 154.94 27.94 0)
+      (effects (font (size 1.27 1.27)) hide)
+    )
+    (pin "1")
+    (pin "2")
+    (instances
+      (project "pcb_xyloauto"
+        (path "/720c51e5-653f-4a9c-b040-f99d22f2970d"
+          (reference "J2") (unit 1)
+        )
+      )
